File: led/led.kicad_pcb (KiCad board)
At the start: 2 copper layers, 13.5 x 16 mm, 3 parts

Commit message: PCB stuff
Parts:
- removed REF**: TerminalBlock_bornier-2_P5.08mm, TerminalBlock:TerminalBlock_bornier-2_P5.08mm
- added J1: Conn_01x02_Female, TerminalBlock:TerminalBlock_bornier-2_P5.08mm, F.Cu at (207.8, 54.9)
Routing:
- net GND: track 8.82 -> 0.00 mm
- added copper zone on F.Cu, net GND
Other:
- outline, holes or cut-outs redrawn
- board text added: "General Kenobi"
- board text added: "Hello there"
Changed lines of the file:
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@@
   (general
     (thickness 1.6)
-    (drawings 5)
-    (tracks 7)
+    (drawings 15)
+    (tracks 4)
     (zones 0)
     (modules 3)
@@
     (34 B.Paste user)
     (35 F.Paste user)
-    (36 B.SilkS user)
+    (36 B.SilkS user hide)
     (37 F.SilkS user)
     (38 B.Mask user)
@@
     (trace_clearance 0.2)
     (zone_clearance 0.508)
-    (zone_45_only no)
+    (zone_45_only yes)
     (trace_min 0.2)
     (via_size 0.8)
@@
   )
   (module TerminalBlock:TerminalBlock_bornier-2_P5.08mm (layer F.Cu)
-    (at 201.93 55.372)
+    (at 207.772 54.864 180)
     (descr "simple 2-pin terminal block, pitch 5.08mm, revamped version of bornier2")
     (tags "terminal block bornier2")
-    (fp_text reference REF** (at 2.54 -5.08) (layer F.SilkS)
-      (effects (font (size 1 1) (thickness 0.15)))
-    )
-    (fp_text value TerminalBlock_bornier-2_P5.08mm (at 2.54 5.08) (layer F.Fab)
+    (fp_text reference J1 (at 2.54 -5.08) (layer F.SilkS)
+      (effects (font (size 1 1) (thickness 0.15)))
+    )
+    (fp_text value Conn_01x02_Female (at 2.54 5.08) (layer F.Fab)
       (effects (font (size 1 1) (thickness 0.15)))
     )
@@
     (fp_line (start 7.79 4) (end 7.79 -4) (layer F.CrtYd) (width 0.05))
     (fp_line (start 7.79 4) (end -2.71 4) (layer F.CrtYd) (width 0.05))
-    (pad 2 thru_hole circle (at 5.08 0) (size 3 3) (drill 1.52) (layers *.Cu *.Mask)
+    (pad 2 thru_hole circle (at 5.08 0 180) (size 3 3) (drill 1.52) (layers *.Cu *.Mask)
+      (net 1 GND))
+    (pad 1 thru_hole rect (at 0 0 180) (size 3 3) (drill 1.52) (layers *.Cu *.Mask)
       (net 3 +5V))
-    (pad 1 thru_hole rect (at 0 0) (size 3 3) (drill 1.52) (layers *.Cu *.Mask)
-      (net 1 GND))
     (model ${KISYS3DMOD}/TerminalBlock.3dshapes/TerminalBlock_bornier-2_P5.08mm.wrl
       (offset (xyz 2.539999961853027 0 0))
@@
       (effects (font (size 1 1) (thickness 0.15)))
     )
+    (fp_line (start 1 -0.6) (end -0.7 -0.6) (layer F.Fab) (width 0.1))
+    (fp_line (start -0.7 -0.6) (end -1 -0.3) (layer F.Fab) (width 0.1))
+    (fp_line (start -1 -0.3) (end -1 0.6) (layer F.Fab) (width 0.1))
+    (fp_line (start -1 0.6) (end 1 0.6) (layer F.Fab) (width 0.1))
+    (fp_line (start 1 0.6) (end 1 -0.6) (layer F.Fab) (width 0.1))
+    (fp_line (start 1 -0.96) (end -1.685 -0.96) (layer F.SilkS) (width 0.12))
+    (fp_line (start -1.685 -0.96) (end -1.685 0.96) (layer F.SilkS) (width 0.12))
+    (fp_line (start -1.685 0.96) (end 1 0.96) (layer F.SilkS) (width 0.12))
+    (fp_line (start -1.68 0.95) (end -1.68 -0.95) (layer F.CrtYd) (width 0.05))
+    (fp_line (start -1.68 -0.95) (end 1.68 -0.95) (layer F.CrtYd) (width 0.05))
+    (fp_line (start 1.68 -0.95) (end 1.68 0.95) (layer F.CrtYd) (width 0.05))
     (fp_line (start 1.68 0.95) (end -1.68 0.95) (layer F.CrtYd) (width 0.05))
-    (fp_line (start 1.68 -0.95) (end 1.68 0.95) (layer F.CrtYd) (width 0.05))
-    (fp_line (start -1.68 -0.95) (end 1.68 -0.95) (layer F.CrtYd) (width 0.05))
-    (fp_line (start -1.68 0.95) (end -1.68 -0.95) (layer F.CrtYd) (width 0.05))
-    (fp_line (start -1.685 0.96) (end 1 0.96) (layer F.SilkS) (width 0.12))
-    (fp_line (start -1.685 -0.96) (end -1.685 0.96) (layer F.SilkS) (width 0.12))
-    (fp_line (start 1 -0.96) (end -1.685 -0.96) (layer F.SilkS) (width 0.12))
-    (fp_line (start 1 0.6) (end 1 -0.6) (layer F.Fab) (width 0.1))
-    (fp_line (start -1 0.6) (end 1 0.6) (layer F.Fab) (width 0.1))
-    (fp_line (start -1 -0.3) (end -1 0.6) (layer F.Fab) (width 0.1))
-    (fp_line (start -0.7 -0.6) (end -1 -0.3) (layer F.Fab) (width 0.1))
-    (fp_line (start 1 -0.6) (end -0.7 -0.6) (layer F.Fab) (width 0.1))
     (fp_text user %R (at 0 0) (layer F.Fab)
       (effects (font (size 0.5 0.5) (thickness 0.08)))
@@
     (tags resistor)
     (attr smd)
-    (fp_text reference R1 (at 0 -1.65) (layer F.SilkS)
-      (effects (font (size 1 1) (thickness 0.15)))
-    )
-    (fp_text value R (at 0 1.65) (layer F.Fab)
-      (effects (font (size 1 1) (thickness 0.15)))
-    )
+    (fp_text reference R1 (at 0 1.737001) (layer F.SilkS)
+      (effects (font (size 1 1) (thickness 0.15)))
+    )
+    (fp_text value R (at 0 -1.818999) (layer F.Fab)
+      (effects (font (size 1 1) (thickness 0.15)))
+    )
+    (fp_line (start -1 0.625) (end -1 -0.625) (layer F.Fab) (width 0.1))
+    (fp_line (start -1 -0.625) (end 1 -0.625) (layer F.Fab) (width 0.1))
+    (fp_line (start 1 -0.625) (end 1 0.625) (layer F.Fab) (width 0.1))
+    (fp_line (start 1 0.625) (end -1 0.625) (layer F.Fab) (width 0.1))
+    (fp_line (start -0.227064 -0.735) (end 0.227064 -0.735) (layer F.SilkS) (width 0.12))
+    (fp_line (start -0.227064 0.735) (end 0.227064 0.735) (layer F.SilkS) (width 0.12))
+    (fp_line (start -1.68 0.95) (end -1.68 -0.95) (layer F.CrtYd) (width 0.05))
+    (fp_line (start -1.68 -0.95) (end 1.68 -0.95) (layer F.CrtYd) (width 0.05))
+    (fp_line (start 1.68 -0.95) (end 1.68 0.95) (layer F.CrtYd) (width 0.05))
     (fp_line (start 1.68 0.95) (end -1.68 0.95) (layer F.CrtYd) (width 0.05))
-    (fp_line (start 1.68 -0.95) (end 1.68 0.95) (layer F.CrtYd) (width 0.05))
-    (fp_line (start -1.68 -0.95) (end 1.68 -0.95) (layer F.CrtYd) (width 0.05))
-    (fp_line (start -1.68 0.95) (end -1.68 -0.95) (layer F.CrtYd) (width 0.05))
-    (fp_line (start -0.227064 0.735) (end 0.227064 0.735) (layer F.SilkS) (width 0.12))
-    (fp_line (start -0.227064 -0.735) (end 0.227064 -0.735) (layer F.SilkS) (width 0.12))
-    (fp_line (start 1 0.625) (end -1 0.625) (layer F.Fab) (width 0.1))
-    (fp_line (start 1 -0.625) (end 1 0.625) (layer F.Fab) (width 0.1))
-    (fp_line (start -1 -0.625) (end 1 -0.625) (layer F.Fab) (width 0.1))
-    (fp_line (start -1 0.625) (end -1 -0.625) (layer F.Fab) (width 0.1))
     (fp_text user %R (at 0 0) (layer F.Fab)
       (effects (font (size 0.5 0.5) (thickness 0.08)))
@@
     )
   )
+  (dimension 16.002 (width 0.15) (layer Dwgs.User)
+    (gr_text "16.002 mm" (at 215.93 51.689 270) (layer Dwgs.User)
+      (effects (font (size 1 1) (thickness 0.15)))
+    )
+    (feature1 (pts (xy 211.328 59.69) (xy 215.216421 59.69)))
+    (feature2 (pts (xy 211.328 43.688) (xy 215.216421 43.688)))
+    (crossbar (pts (xy 214.63 43.688) (xy 214.63 59.69)))
+    (arrow1a (pts (xy 214.63 59.69) (xy 214.043579 58.563496)))
+    (arrow1b (pts (xy 214.63 59.69) (xy 215.216421 58.563496)))
+    (arrow2a (pts (xy 214.63 43.688) (xy 214.043579 44.814504)))
+    (arrow2b (pts (xy 214.63 43.688) (xy 215.216421 44.814504)))
+  )
+  (dimension 13.462 (width 0.15) (layer Dwgs.User)
+    (gr_text "13.462 mm" (at 204.597 39.848) (layer Dwgs.User)
+      (effects (font (size 1 1) (thickness 0.15)))
+    )
+    (feature1 (pts (xy 211.328 43.688) (xy 211.328 40.561579)))
+    (feature2 (pts (xy 197.866 43.688) (xy 197.866 40.561579)))
+    (crossbar (pts (xy 197.866 41.148) (xy 211.328 41.148)))
+    (arrow1a (pts (xy 211.328 41.148) (xy 210.201496 41.734421)))
+    (arrow1b (pts (xy 211.328 41.148) (xy 210.201496 40.561579)))
+    (arrow2a (pts (xy 197.866 41.148) (xy 198.992504 41.734421)))
+    (arrow2b (pts (xy 197.866 41.148) (xy 198.992504 40.561579)))
+  )
+  (gr_text "General Kenobi" (at 199.136 50.038 90) (layer B.SilkS)
+    (effects (font (size 1 1) (thickness 0.15)) (justify mirror))
+  )
+  (gr_text "Hello there" (at 199.136 48.514 90) (layer F.SilkS)
+    (effects (font (size 1 1) (thickness 0.15)))
+  )
+  (gr_line (start 198.12 59.436) (end 198.12 43.942) (layer F.SilkS) (width 0.12))
+  (gr_line (start 211.074 59.436) (end 198.12 59.436) (layer F.SilkS) (width 0.12))
+  (gr_line (start 211.074 43.942) (end 211.074 59.436) (layer F.SilkS) (width 0.12))
+  (gr_line (start 208.28 43.942) (end 211.074 43.942) (layer F.SilkS) (width 0.12))
+  (gr_line (start 198.12 43.942) (end 208.28 43.942) (layer F.SilkS) (width 0.12))
+  (gr_circle (center 209.804 44.958) (end 210.312 44.45) (layer Edge.Cuts) (width 0.05))
   (gr_line (start 211.328 43.688) (end 197.866 43.688) (layer Edge.Cuts) (width 0.05))
   (gr_circle (center 205.01 50.292) (end 207.01 50.292) (layer Edge.Cuts) (width 0.05))
@@
   (gr_line (start 211.328 59.69) (end 197.866 59.69) (layer Edge.Cuts) (width 0.05))
   (gr_line (start 211.328 43.688) (end 211.328 59.69) (layer Edge.Cuts) (width 0.05))
-  (segment (start 201.93 55.372) (end 201.93 50.292) (width 0.25) (layer F.Cu) (net 1))
-  (segment (start 201.467501 49.829501) (end 201.467501 46.740001) (width 0.25) (layer F.Cu) (net 1))
-  (segment (start 201.93 50.292) (end 201.467501 49.829501) (width 0.25) (layer F.Cu) (net 1))
   (segment (start 205.857501 46.740001) (end 205.902501 46.695001) (width 0.25) (layer F.Cu) (net 2))
   (segment (start 203.342501 46.740001) (end 205.857501 46.740001) (width 0.25) (layer F.Cu) (net 2))
-  (segment (start 207.727501 54.654499) (end 207.01 55.372) (width 0.25) (layer F.Cu) (net 3))
-  (segment (start 207.727501 46.695001) (end 207.727501 54.654499) (width 0.25) (layer F.Cu) (net 3))
+  (segment (start 208.788 47.7555) (end 208.788 54.864) (width 0.25) (layer F.Cu) (net 3))
+  (segment (start 207.727501 46.695001) (end 208.788 47.7555) (width 0.25) (layer F.Cu) (net 3))
+  (zone (net 1) (net_name GND) (layer F.Cu) (hatch edge 0.508)
+    (connect_pads (clearance 0.508))
+    (min_thickness 0.254)
+    (fill yes (arc_segments 32) (thermal_gap 0.508) (thermal_bridge_width 0.508))
+    (polygon
+      (pts
+        (xy 211.074 59.436) (xy 198.12 59.436) (xy 198.12 43.942) (xy 211.074 43.942)
+      )
+    )
+  )
 )
