File: arduino/arduino.kicad_pcb (KiCad board)
At the start: 2 copper layers, 17 parts, among them J1 Digital pins, J2 ICSP, J3 I2C, J4 SERIAL, U1 ATmega328P-AU, U2 24LC1025, U3 DS1337, U4 24LC1025, Y1 32,768MHz, Y2 16MHz

Commit message: Finish course
Parts:
- moved R1 19.1 mm to (149.5, 130.2)
- moved C1 18.2 mm to (130.2, 124.2), turned to 180 degrees
- moved C2 17.8 mm to (130.2, 128.1), turned to 180 degrees
- moved D1 15.1 mm to (151.0, 126.9), turned to 270 degrees
- moved R2 13.7 mm to (141.9, 112.4)
- moved U3 11.6 mm to (133.8, 117.8)
- moved Y1 11.4 mm to (131.1, 112.4)
- moved U1 8.07 mm to (144.6, 120.6), turned to 0 degrees
- moved Y2 7.82 mm to (134.0, 126.1), turned to 90 degrees
- moved C3 7.80 mm to (125.0, 118.4)
- moved J3 5.87 mm to (140.9, 107.8)
- moved BT1 2.95 mm to (122.9, 110.2)
- moved J4 2.40 mm to (136.5, 107.8)
Connections:
- U1 pad 23: /ADDS1 -> /ADDS2
- U1 pad 24: /ADDS2 -> /ADDS1
Other:
- board outline added: 38.3 x 29.8 mm
